Commit message: Diseño de robot - Links y joints establecidas

File: differential_robot_description/urdf/diff_segismundo.urdf (robot description, URDF)
Before this commit: robot diff_segismundo, 1 links, 0 joints
Links:
- added link base_footprint
- added link caster_wheel_link; visual sphere radius=0.05
- added link left_wheel_link; visual cylinder length=0.05 radius=0.1
- added link right_wheel_link; visual cylinder length=0.05 radius=0.1
- link base_link: geometry visual box size=0.6 0.4 0.2
Joints:
- added joint base_to_caster_wheel: type continuous, parent base_link, child caster_wheel_link, origin xyz=0.2 0.0 -0.05 rpy=0.0 0.0 0.0, axis 0.0 1.0 0.0
- added joint base_to_left_wheel: type continuous, parent base_link, child left_wheel_link, origin xyz=-0.15 0.225 0.0 rpy=0.0 0.0 0.0, axis 0.0 1.0 0.0
- added joint base_to_right_wheel: type continuous, parent base_link, child right_wheel_link, origin xyz=-0.15 -0.225 0.0 rpy=0.0 0.0 0.0, axis 0.0 1.0 0.0
- added joint footprint_to_base_joint: type fixed, parent base_footprint, child base_link, origin xyz=0.0 0.0 0.1 rpy=0.0 0.0 0.0
