Commit message: GZ SIM - Paquete differential_robot_bringup creado - Launch implementado con los nodos para lanzar gz sim y rviz - Plugins para diff-drive system y para joint state publisher obtenidos de https://github.com/gazebosim/gz-sim/tree/gz-sim9/src

File: differential_robot_description/urdf/diff_segismundo.urdf.xacro (robot description, xacro)
@@ -3,4 +3,5 @@
     <xacro:include filename="$(find differential_robot_description)/urdf/common_properties.xacro" />
     <xacro:include filename="$(find differential_robot_description)/urdf/mobile_base.xacro" />
+    <xacro:include filename="$(find differential_robot_description)/urdf/mobile_base_gazebo.xacro" />
     <!-- UBUNTU 24-->
 </robot>

File: differential_robot_description/urdf/mobile_base.xacro (robot description, xacro)
@@ -94,5 +94,5 @@
         <axis xyz="0.0 1.0 0.0"/>
     </joint>
-    <joint name="base_to_caster_wheel" type="continuous">
+    <joint name="base_to_caster_wheel" type="fixed">
         <parent link="base_link"/>
         <child link="caster_wheel_link"/>
