Commit message: Gazebo
Colision e intercia implementadas en los eslabones para su visualización en Gazebo

File: differential_robot_description/urdf/common_properties.xacro (robot description, xacro)
@@ -10,3 +10,30 @@
         <color rgba="0.0 .0 0.0 1.0"/>
     </material>
+    <xacro:macro name="box_inertia" params="l w h m o_xyz o_rpy">
+      <inertial>
+        <origin xyz="${o_xyz}" rpy="${o_rpy}"/>
+        <mass value="${m}"/>
+        <inertia ixx="${m*(w*w+h*h)/12.0}" ixy="0.0" ixz="0.0"
+                 iyy="${m*(l*l+h*h)/12.0}" iyz="0.0"
+                 izz="${m*(w*w+l*l)/12.0}"/>
+      </inertial>
+    </xacro:macro>
+    <xacro:macro name="cylinder_inertia" params="r l m o_xyz o_rpy">
+      <inertial>
+        <origin xyz="${o_xyz}" rpy="${o_rpy}"/>
+        <mass value="${m}"/>
+        <inertia ixx="${m*(3*r*r+l*l)/12.0}" ixy="0.0" ixz="0.0"
+                 iyy="${m*(l*l+3*r*r)/12.0}" iyz="0.0"
+                 izz="${m*(r*r)/2.0}"/>
+      </inertial>
+    </xacro:macro>
+    <xacro:macro name="sphere_inertia" params="r m o_xyz o_rpy">
+      <inertial>
+        <origin xyz="${o_xyz}" rpy="${o_rpy}"/>
+        <mass value="${m}"/>
+        <inertia ixx="${2*m*r*r/5.0}" ixy="0.0" ixz="0.0"
+                 iyy="${2*m*r*r/5.0}" iyz="0.0"
+                 izz="${2*m*r*r/5.0}"/>
+      </inertial>
+    </xacro:macro>
 </robot>

File: differential_robot_description/urdf/mobile_base.xacro (robot description, xacro)
@@ -8,22 +8,36 @@
     <xacro:macro name="wheel_link" params="prefix radius length">
         <link name="${prefix}_wheel_link">
-        <visual>
-            <geometry>
-                <cylinder radius="${radius}" length="${length}"/>
-            </geometry>
-            <origin xyz="0.0 0.0 0.0" rpy="${pi / 2.0} 0.0 0.0"/>
-            <material name="grey"/>
-        </visual>
-    </link>
+            <xacro:cylinder_inertia r="${wheel_radius}" l="${wheel_length}" m="1.0" o_xyz="0.0 0.0 0.0" o_rpy="${pi / 2.0} 0.0 0.0"/>
+            <visual>
+                <geometry>
+                    <cylinder radius="${wheel_radius}" length="${wheel_length}"/>
+                </geometry>
+                <origin xyz="0.0 0.0 0.0" rpy="${pi / 2.0} 0.0 0.0"/>
+                <material name="grey"/>
+            </visual>
+            <collision>
+                <geometry>
+                    <sphere radius="${wheel_radius}"/>
+                </geometry>
+                <origin xyz="0.0 0.0 0.0" rpy="${pi / 2.0} 0.0 0.0"/>
+            </collision>
+        </link>
     </xacro:macro>
     <link name="base_footprint"></link>
     <link name="base_link">
+        <xacro:box_inertia l="${base_length}" w="${base_width}" h="${base_height}" m="5.0" o_xyz="0.0 0.0 ${wheel_radius}" o_rpy="0.0 0.0 0.0"/>
         <visual>
             <geometry>
                 <box size="${base_length} ${base_width} ${base_height}"/>
             </geometry>
-            <origin xyz="0.0 0.0 ${wheel_radius}" rpy="0.0 0.0 0.0"/>
+            <origin xyz="0.0 0.0 ${base_height/2}" rpy="0.0 0.0 0.0"/>
             <material name="blue"/>
         </visual>
+        <collision>
+            <geometry>
+                <box size="${base_length} ${base_width} ${base_height}"/>
+            </geometry>
+            <origin xyz="0.0 0.0 ${base_height/2}" rpy="0.0 0.0 0.0"/>
+        </collision>
     </link>
     <!-- <link name="right_wheel_link">
@@ -48,4 +62,5 @@
     </link> -->
     <link name="caster_wheel_link">
+        <xacro:sphere_inertia r="${wheel_radius/2}" m="0.5" o_xyz="0.0 0.0 0.0" o_rpy="0.0 0.0 0.0"/>
         <visual>
             <geometry>
@@ -55,4 +70,10 @@
             <material name="grey"/>
         </visual>
+        <collision>
+            <geometry>
+                <sphere radius="${wheel_radius / 2}"/>
+            </geometry>
+            <origin xyz="0.0 0.0 0.0" rpy="0 0.0 0.0"/>
+        </collision>
     </link>
     <joint name="footprint_to_base_joint" type="fixed">

Commit message: NUEVOS MATERIALES - Nuevos colores de materiales implementados

File: differential_robot_description/urdf/common_properties.xacro (robot description, xacro)
@@ -9,4 +9,13 @@
     <material name="black">
         <color rgba="0.0 .0 0.0 1.0"/>
+    </material>
+    <material name="aquagreen" >
+        <color rgba="0.07058823529411765 0.8823529411764706 0.5764705882352941 1.0" />
+    </material>
+    <material name="amber" >
+        <color rgba="0.996078431372549 0.7019607843137254 0.03137254901960784 1.0" />
+    </material>
+    <material name="bluegrey" >
+        <color rgba="0.5215686274509804 0.6392156862745098 0.6980392156862745 1.0" />
     </material>
     <xacro:macro name="box_inertia" params="l w h m o_xyz o_rpy">
