Commit message: NAV2 AUTÓNOMA
- navegación autónoma en el mapa implementada
- pkg de navegación creado

File: hack_pue_2025/hera_robot_description/urdf/mobile_base.xacro (robot description, xacro)
@@ -18,5 +18,6 @@
             <collision>
                 <geometry>
-                    <sphere radius="${wheel_radius}"/>
+                    <!-- <sphere radius="${wheel_radius}"/> -->
+                    <cylinder radius="${wheel_radius}" length="${wheel_length}"/>
                 </geometry>
                 <origin xyz="0.0 0.0 0.0" rpy="${pi / 2.0} 0.0 0.0"/>

Commit message: MAPPING ACTUALIZADO
- Reconfiguración del mundo
- Remapeo para la simulación de navegación autónoma

File: hack_pue_2025/hera_robot_description/urdf/mobile_base.xacro (robot description, xacro)
@@ -18,6 +18,5 @@
             <collision>
                 <geometry>
-                    <!-- <sphere radius="${wheel_radius}"/> -->
-                    <cylinder radius="${wheel_radius}" length="${wheel_length}"/>
+                    <sphere radius="${wheel_radius}"/>
                 </geometry>
                 <origin xyz="0.0 0.0 0.0" rpy="${pi / 2.0} 0.0 0.0"/>
