Commit message: CAMERA & MATERIALS - Cámara con visión artificial implementada - Configuración de ign gazebo y de rviz actualizadas - Nuevos materiales añadidos a mobile_base

File: hack_pue_2025/hera_robot_description/urdf/common_properties.xacro (robot description, xacro)
@@ -18,4 +18,19 @@
     <material name="bluegrey" >
         <color rgba="0.5215686274509804 0.6392156862745098 0.6980392156862745 1.0" />
+    </material>
+    <material name="lime">
+        <color rgba="0.7647 0.9686 0.2275 1.0"/>
+    </material>
+    <material name="light_green">
+        <color rgba="0.5843 0.8784 0.4235 1.0"/>
+    </material>
+    <material name="mint">
+        <color rgba="0.4078 0.7137 0.5176 1.0"/>
+    </material>
+    <material name="polynesian_blue">
+        <color rgba="0.0353 0.3020 0.5725 1.0"/>
+    </material>
+    <material name="licorice">
+        <color rgba="0.1098 0.0627 0.0941 1.0"/>
     </material>
     <xacro:macro name="box_inertia" params="l w h m o_xyz o_rpy">

File: hack_pue_2025/hera_robot_description/urdf/diff_hera.urdf.xacro (robot description, xacro)
@@ -4,5 +4,5 @@
     <xacro:include filename="$(find hera_robot_description)/urdf/mobile_base.xacro" />
     <xacro:include filename="$(find hera_robot_description)/urdf/mobile_base_gazebo.xacro" />
-    <!-- <xacro:include filename="$(find hera_robot_description)/urdf/camera.xacro" /> -->
+    <xacro:include filename="$(find hera_robot_description)/urdf/camera.xacro" />
     <xacro:include filename="$(find hera_robot_description)/urdf/lidar.xacro" />
     <!-- UBUNTU 24-->

File: hack_pue_2025/hera_robot_description/urdf/lidar.xacro (robot description, xacro)
@@ -11,5 +11,5 @@
                 <cylinder radius="${lidar_radius}" length="${lidar_length}"/>
             </geometry>
-            <material name="bluegrey"/>
+            <material name="polynesian_blue"/>
         </visual>
         <collision>
@@ -53,7 +53,4 @@
                 </noise>
             </lidar>
-            <plugin filename="gz-sim-sensors-system" name="gz::sim::systems::Sensors">
-                <render_engine>ogre2</render_engine>
-            </plugin>
         </sensor>
     </gazebo>

File: hack_pue_2025/hera_robot_description/urdf/mobile_base.xacro (robot description, xacro)
@@ -14,5 +14,5 @@
                 </geometry>
                 <origin xyz="0.0 0.0 0.0" rpy="${pi / 2.0} 0.0 0.0"/>
-                <material name="grey"/>
+                <material name="licorice"/>
             </visual>
             <collision>
@@ -32,5 +32,5 @@
             </geometry>
             <origin xyz="0.0 0.0 ${base_height/2}" rpy="0.0 0.0 0.0"/>
-            <material name="blue"/>
+            <material name="mint"/>
         </visual>
         <collision>
@@ -50,5 +50,5 @@
             </geometry>
             <origin xyz="0.0 0.0 0.0" rpy="0 0.0 0.0"/>
-            <material name="grey"/>
+            <material name="licorice"/>
         </visual>
         <collision>
